File: BMS.kicad_sch (KiCad schematic)
At the start: 80 parts, among them J1 Screw_Terminal_01x02, J5 BATT_PACK -, Q22 CSD19531Q5A, Q23 CSD19531Q5A, Q24 CSD19531Q5A, T3 EE20_10_6_750811647, U1 TL431DBZ, U18 VIPer26LD, U2 PC817, U21 BQ7790500PWR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

Commit message: Routing update
 19 errors to go
Parts:
- RV1: footprint (none) -> Resistor_SMD:R_0805_2012Metric
- RV2, RV3: footprint (none) -> Potentiometer_SMD:Potentiometer_ACP_CA6-VSMD_Vertical
Changed lines of the file:
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@@
 	)
 	(junction
-		(at 261.62 177.8)
-		(diameter 0)
-		(color 0 0 0 0)
-	)
-	(junction
 		(at 127 76.2)
 		(diameter 0)
@@
 	)
 	(junction
+		(at 261.62 177.8)
+		(diameter 0)
+		(color 0 0 0 0)
+	)
+	(junction
 		(at 73.66 233.68)
 		(diameter 0)
@@
 	(wire
 		(pts
+			(xy 261.62 177.8) (xy 280.67 177.8)
+		)
+		(stroke
+			(width 0)
+			(type default)
+		)
+	)
+	(wire
+		(pts
 			(xy 138.43 180.34) (xy 152.4 180.34)
 		)
@@
 	(wire
 		(pts
-			(xy 261.62 177.8) (xy 280.67 177.8)
+			(xy 245.11 177.8) (xy 261.62 177.8)
 		)
 		(stroke
@@
 	(wire
 		(pts
+			(xy 261.62 160.02) (xy 261.62 177.8)
+		)
+		(stroke
+			(width 0)
+			(type default)
+		)
+	)
+	(wire
+		(pts
 			(xy 217.17 220.98) (xy 226.06 220.98)
 		)
@@
 	(wire
 		(pts
-			(xy 245.11 177.8) (xy 261.62 177.8)
-		)
-		(stroke
-			(width 0)
-			(type default)
-		)
-	)
-	(wire
-		(pts
 			(xy 39.37 54.61) (xy 41.91 54.61)
 		)
@@
 	(wire
 		(pts
-			(xy 261.62 177.8) (xy 261.62 181.61)
-		)
-		(stroke
-			(width 0)
-			(type default)
-		)
-	)
-	(wire
-		(pts
 			(xy 212.09 39.37) (xy 224.79 39.37)
 		)
@@
 	(wire
 		(pts
-			(xy 261.62 160.02) (xy 261.62 177.8)
-		)
-		(stroke
-			(width 0)
-			(type default)
-		)
-	)
-	(wire
-		(pts
 			(xy 38.1 158.75) (xy 50.8 158.75)
 		)
@@
 		)
 	)
-	(global_label "V-"
-		(shape input)
-		(at 261.62 181.61 270)
-		(fields_autoplaced yes)
-		(effects
-			(font
-				(size 1.27 1.27)
-			)
-			(justify right)
-		)
-		(property "Intersheetrefs" "${INTERSHEET_REFS}"
-			(at 261.62 187.2562 90)
-			(hide yes)
-			(show_name no)
-			(do_not_autoplace no)
-			(effects
-				(font
-					(size 1.27 1.27)
-				)
-				(justify right)
-			)
-		)
-	)
 	(global_label "VO"
 		(shape output)
@@
 			)
 		)
-		(property "Footprint" ""
+		(property "Footprint" "Potentiometer_SMD:Potentiometer_ACP_CA6-VSMD_Vertical"
 			(at 379.73 170.18 0)
 			(hide yes)
@@
 		(lib_id "Device:R")
 		(at 205.74 154.94 0)
+		(mirror y)
 		(unit 1)
 		(body_style 1)
@@
 		(dnp no)
 		(property "Reference" "R1"
-			(at 203.708 154.94 90)
+			(at 207.772 154.94 90)
 			(show_name no)
 			(do_not_autoplace no)
@@
 		)
 		(property "Value" "220Ohm"
-			(at 209.55 154.94 90)
+			(at 201.93 154.94 90)
 			(show_name no)
 			(do_not_autoplace no)
@@
 		)
 		(property "Footprint" "Resistor_SMD:R_0805_2012Metric"
-			(at 203.962 154.94 90)
+			(at 207.518 154.94 90)
 			(hide yes)
 			(show_name no)
@@
 			)
 		)
-		(property "Footprint" ""
+		(property "Footprint" "Resistor_SMD:R_0805_2012Metric"
 			(at 361.95 177.8 0)
 			(hide yes)
@@
 			)
 		)
-		(property "Footprint" ""
+		(property "Footprint" "Potentiometer_SMD:Potentiometer_ACP_CA6-VSMD_Vertical"
 			(at 358.14 148.59 0)
 			(hide yes)
@@
 		(lib_id "Device:C_Polarized")
 		(at 224.79 50.8 0)
+		(mirror y)
 		(unit 1)
 		(body_style 1)
@@
 		(dnp no)
 		(property "Reference" "C2"
-			(at 225.806 47.244 0)
+			(at 223.774 47.244 0)
 			(show_name no)
 			(do_not_autoplace no)
@@
 		)
 		(property "Value" "470uF"
-			(at 225.806 54.356 0)
+			(at 223.774 54.356 0)
 			(show_name no)
 			(do_not_autoplace no)
@@
 		)
 		(property "Footprint" "Capacitor_SMD:C_0805_2012Metric"
-			(at 225.7552 54.61 0)
+			(at 223.8248 54.61 0)
 			(hide yes)
 			(show_name no)
